Commit message: changes for moveit

File: urdf/prbt.xacro (robot description, xacro)
@@ -1,56 +1,24 @@
-<?xml version="1.0" encoding="utf-8" ?>
-<!--
-Copyright (c) 2018 Pilz GmbH & Co. KG
-Licensed under the Apache License, Version 2.0 (the "License");
-you may not use this file except in compliance with the License.
-You may obtain a copy of the License at
-    http://www.apache.org/licenses/LICENSE-2.0
-Unless required by applicable law or agreed to in writing, software
-distributed under the License is distributed on an "AS IS" BASIS,
-WITHOUT WARRANTIES OR CONDITIONS OF ANY KIND, either express or implied.
-See the License for the specific language governing permissions and
-limitations under the License.
--->
-<robot name="prbt" xmlns:xacro="http://www.ros.org/wiki/xacro">
-  <!-- Definition of robot name -->
+<?xml version="1.0"?>
+<robot xmlns:xacro="http://www.ros.org/wiki/xacro" name="prbt">
   <xacro:arg name="robot_prefix" default="prbt_"/>
-  <!-- macro definition of pilz lwa -->
+  <xacro:arg name="bus_config" default="$(find prbt_robot)/config/prbt/bus.yml"/>
+  <xacro:arg name="master_config" default="$(find prbt_robot)/config/prbt/master.dcf"/>
+  <xacro:arg name="can_interface" default="vcan0"/>
+  <xacro:arg name="master_bin" default=""/>
+  <xacro:include filename="$(find prbt_robot)/urdf/prbt.ros2_control.xacro" />
   <xacro:include filename="$(find prbt_robot)/urdf/prbt_macro.xacro" />
-  <!-- gripper -->
-  <xacro:arg name="gripper" default=""/>
-  <xacro:property name="gripper" value="$(arg gripper)"/>
+  <xacro:prbt_ros2_control name="prbt" prefix="$(arg robot_prefix)" bus_config="$(arg bus_config)" master_config="$(arg master_config)" can_interface="$(arg can_interface)" master_bin="$(arg master_bin)" />
   <!-- TCP Offset -->
-  <xacro:if value="${not gripper}">
-    <xacro:arg name="tcp_offset_xyz" default="0 0 0"/>
-    <xacro:arg name="tcp_offset_rpy" default="0 0 0"/>
-  </xacro:if>
-  <xacro:if value="${gripper != ''}">
-    <xacro:include filename="$(find prbt_${gripper}_support)/config/${gripper}_tcp_offset.xacro" />
-  </xacro:if>
+  <xacro:arg name="tcp_offset_xyz" default="0 0 0"/>
+  <xacro:arg name="tcp_offset_rpy" default="0 0 0"/>
   <!-- instantiate the robot -->
   <xacro:prbt prefix="$(arg robot_prefix)" />
-  <link name="world"/>
-  <joint name="world-base_link-fixed" type="fixed">
-    <parent link="world"/>
-    <child link="$(arg robot_prefix)base_link"/>
-  </joint>
   <!-- TCP -->
   <joint name="$(arg robot_prefix)fixed_joint_tcp" type="fixed">
-    <origin xyz="$(arg tcp_offset_xyz)" rpy="$(arg tcp_offset_rpy)" />  <!-- tcp offset from last link -->
+    <origin xyz="$(arg tcp_offset_xyz)" rpy="$(arg tcp_offset_rpy)" />
+    <!-- tcp offset from last link -->
     <parent link="$(arg robot_prefix)flange"/>
     <child link="$(arg robot_prefix)tcp"/>
   </joint>
   <link name="$(arg robot_prefix)tcp" />
-  <!-- If gripper given then... -->
-  <xacro:if value="${gripper != ''}">
-    <!-- name of the gripper -->
-    <xacro:property name="gripper_name" value="$(arg robot_prefix)gripper"/>
-    <!-- load gripper macro -->
-    <xacro:include filename="$(find prbt_${gripper}_support)/urdf/${gripper}.urdf.xacro" />
-    <!-- instantiate gripper -->
-    <xacro:prbt_gripper parent="$(arg robot_prefix)flange" />
-    <!-- Add gripper brackets -->
-    <xacro:include filename="$(find prbt_support)/urdf/simple_gripper_brackets.urdf.xacro" />
-    <xacro:simple_gripper_brackets />
-  </xacro:if>
 </robot>

File: urdf/prbt_macro.xacro (robot description, xacro)
@@ -1,15 +1,3 @@
-<?xml version="1.0" encoding="utf-8" ?>
-<!--
-Copyright (c) 2018 Pilz GmbH & Co. KG
-Licensed under the Apache License, Version 2.0 (the "License");
-you may not use this file except in compliance with the License.
-You may obtain a copy of the License at
-    http://www.apache.org/licenses/LICENSE-2.0
-Unless required by applicable law or agreed to in writing, software
-distributed under the License is distributed on an "AS IS" BASIS,
-WITHOUT WARRANTIES OR CONDITIONS OF ANY KIND, either express or implied.
-See the License for the specific language governing permissions and
-limitations under the License.
--->
+<?xml version="1.0"?>
 <robot xmlns:xacro="http://www.ros.org/wiki/xacro">
   <xacro:macro name="prbt" params="prefix">
@@ -24,8 +12,8 @@
     <!-- robot foot link -->
     <link name="${prefix}base_link">
-        <inertial>
-          <mass value="2.4"/>
-          <inertia ixx="0"  ixy="0"  ixz="0" iyy="0" iyz="0" izz="0" />
-        </inertial>
+      <inertial>
+        <mass value="2.4"/>
+        <inertia ixx="0" ixy="0" ixz="0" iyy="0" iyz="0" izz="0" />
+      </inertial>
       <visual>
         <origin xyz="0 0 0" rpy="0 0 0" />
@@ -95,5 +83,5 @@
         <mass value="1.7"/>
         <origin xyz="0 0.162 0.134" />
-        <inertia ixx="3.58e-2"  ixy="0"  ixz="0" iyy="3.22e-3" iyz="-1.45e-3" izz="3.66e-2" />
+        <inertia ixx="3.58e-2" ixy="0" ixz="0" iyy="3.22e-3" iyz="-1.45e-3" izz="3.66e-2" />
       </inertial>
       <visual name="first">
@@ -329,8 +317,8 @@
     </transmission>
     <gazebo>
-      <plugin name="gazebo_ros_control" filename="libgazebo_ros_control.so" >
+      <plugin name="gazebo_ros_control" filename="libgazebo_ros_control.so">
         <robotNamespace>prbt</robotNamespace>
         <robotSimType>gazebo_ros_control/DefaultRobotHWSim</robotSimType>
-        <legacyModeNS>false</legacyModeNS> <!-- Only used from ros-kinetic-gazebo-ros-control 2.5.18 -->
+        <legacyModeNS>false</legacyModeNS>        <!-- Only used from ros-kinetic-gazebo-ros-control 2.5.18 -->
       </plugin>
     </gazebo>
@@ -340,7 +328,7 @@
     <gazebo>
       <plugin name="ft_sensor" filename="libgazebo_ros_ft_sensor.so">
-	<updateRate>100.0</updateRate>
-	<topicName>prbt/ft_sensor/joint_1</topicName>
-	<jointName>${prefix}joint_1</jointName>
+        <updateRate>100.0</updateRate>
+        <topicName>prbt/ft_sensor/joint_1</topicName>
+        <jointName>${prefix}joint_1</jointName>
       </plugin>
     </gazebo>
@@ -350,7 +338,7 @@
     <gazebo>
       <plugin name="ft_sensor" filename="libgazebo_ros_ft_sensor.so">
-	<updateRate>100.0</updateRate>
-	<topicName>prbt/ft_sensor/joint_2</topicName>
-	<jointName>${prefix}joint_2</jointName>
+        <updateRate>100.0</updateRate>
+        <topicName>prbt/ft_sensor/joint_2</topicName>
+        <jointName>${prefix}joint_2</jointName>
       </plugin>
     </gazebo>
@@ -360,7 +348,7 @@
     <gazebo>
       <plugin name="ft_sensor" filename="libgazebo_ros_ft_sensor.so">
-	<updateRate>100.0</updateRate>
-	<topicName>prbt/ft_sensor/joint_3</topicName>
-	<jointName>${prefix}joint_3</jointName>
+        <updateRate>100.0</updateRate>
+        <topicName>prbt/ft_sensor/joint_3</topicName>
+        <jointName>${prefix}joint_3</jointName>
       </plugin>
     </gazebo>
@@ -370,7 +358,7 @@
     <gazebo>
       <plugin name="ft_sensor" filename="libgazebo_ros_ft_sensor.so">
-	<updateRate>100.0</updateRate>
-	<topicName>prbt/ft_sensor/joint_4</topicName>
-	<jointName>${prefix}joint_4</jointName>
+        <updateRate>100.0</updateRate>
+        <topicName>prbt/ft_sensor/joint_4</topicName>
+        <jointName>${prefix}joint_4</jointName>
       </plugin>
     </gazebo>
@@ -380,7 +368,7 @@
     <gazebo>
       <plugin name="ft_sensor" filename="libgazebo_ros_ft_sensor.so">
-	<updateRate>100.0</updateRate>
-	<topicName>prbt/ft_sensor/joint_5</topicName>
-	<jointName>${prefix}joint_5</jointName>
+        <updateRate>100.0</updateRate>
+        <topicName>prbt/ft_sensor/joint_5</topicName>
+        <jointName>${prefix}joint_5</jointName>
       </plugin>
     </gazebo>
@@ -390,7 +378,7 @@
     <gazebo>
       <plugin name="ft_sensor" filename="libgazebo_ros_ft_sensor.so">
-	<updateRate>100.0</updateRate>
-	<topicName>prbt/ft_sensor/joint_6</topicName>
-	<jointName>${prefix}joint_6</jointName>
+        <updateRate>100.0</updateRate>
+        <topicName>prbt/ft_sensor/joint_6</topicName>
+        <jointName>${prefix}joint_6</jointName>
       </plugin>
     </gazebo>
