Commit message: Add moveit config and restructure

File: prbt_robot_support/urdf/prbt.xacro (robot description, xacro)
@@ -2,10 +2,10 @@
 <robot xmlns:xacro="http://www.ros.org/wiki/xacro" name="prbt">
   <xacro:arg name="robot_prefix" default="prbt_"/>
-  <xacro:arg name="bus_config" default="$(find prbt_robot)/config/prbt/bus.yml"/>
-  <xacro:arg name="master_config" default="$(find prbt_robot)/config/prbt/master.dcf"/>
+  <xacro:arg name="bus_config" default="$(find prbt_robot_support)/config/prbt/bus.yml"/>
+  <xacro:arg name="master_config" default="$(find prbt_robot_support)/config/prbt/master.dcf"/>
   <xacro:arg name="can_interface" default="vcan0"/>
   <xacro:arg name="master_bin" default=""/>
-  <xacro:include filename="$(find prbt_robot)/urdf/prbt.ros2_control.xacro" />
-  <xacro:include filename="$(find prbt_robot)/urdf/prbt_macro.xacro" />
+  <xacro:include filename="$(find prbt_robot_support)/urdf/prbt.ros2_control.xacro" />
+  <xacro:include filename="$(find prbt_robot_support)/urdf/prbt_macro.xacro" />
   <xacro:prbt_ros2_control name="prbt" prefix="$(arg robot_prefix)" bus_config="$(arg bus_config)" master_config="$(arg master_config)" can_interface="$(arg can_interface)" master_bin="$(arg master_bin)" />
   <!-- TCP Offset -->

File: prbt_robot_support/urdf/prbt_macro.xacro (robot description, xacro)
@@ -19,5 +19,5 @@
         <origin xyz="0 0 0" rpy="0 0 0" />
         <geometry>
-          <mesh filename="package://prbt_robot/meshes/foot.dae" />
+          <mesh filename="package://prbt_robot_support/meshes/foot.dae" />
         </geometry>
       </visual>
@@ -48,5 +48,5 @@
         <origin xyz="0 0 0" rpy="0 0 0" />
         <geometry>
-          <mesh filename="package://prbt_robot/meshes/link_1.dae" />
+          <mesh filename="package://prbt_robot_support/meshes/link_1.dae" />
         </geometry>
       </visual>
@@ -88,5 +88,5 @@
         <origin xyz="0 0 0" rpy="0 0 0" />
         <geometry>
-          <mesh filename="package://prbt_robot/meshes/link_2.dae" />
+          <mesh filename="package://prbt_robot_support/meshes/link_2.dae" />
         </geometry>
       </visual>
@@ -122,5 +122,5 @@
         <origin xyz="0 0 0" rpy="0 0 0" />
         <geometry>
-          <mesh filename="package://prbt_robot/meshes/link_3.dae" />
+          <mesh filename="package://prbt_robot_support/meshes/link_3.dae" />
         </geometry>
       </visual>
@@ -162,5 +162,5 @@
         <origin xyz="0 0 0" rpy="0 0 0" />
         <geometry>
-          <mesh filename="package://prbt_robot/meshes/link_4.dae" />
+          <mesh filename="package://prbt_robot_support/meshes/link_4.dae" />
         </geometry>
       </visual>
@@ -196,5 +196,5 @@
         <origin xyz="0 0 0" rpy="0 0 0" />
         <geometry>
-          <mesh filename="package://prbt_robot/meshes/link_5.dae"/>
+          <mesh filename="package://prbt_robot_support/meshes/link_5.dae"/>
         </geometry>
       </visual>
@@ -249,5 +249,5 @@
         <origin xyz="0 0 0" rpy="0 0 0" />
         <geometry>
-          <mesh filename="package://prbt_robot/meshes/flange.dae"/>
+          <mesh filename="package://prbt_robot_support/meshes/flange.dae"/>
         </geometry>
       </visual>
