Commit message: Minor fix to launch files and xacro files

File: prbt_robot_moveit_config/config/prbt.ros2_control.xacro (robot description, xacro)
@@ -9,5 +9,5 @@
       master_bin
       initial_positions_file">
-    <xacro:property name="initial_positions" value="${load_yaml(initial_positions_file)['initial_positions']}"/>
+    <xacro:property name="initial_positions" value="${xacro.load_yaml(initial_positions_file)['initial_positions']}"/>
     <ros2_control name="${name}" type="system">
       <hardware>

File: prbt_robot_support/urdf/prbt.xacro (robot description, xacro)
@@ -1,24 +1,18 @@
 <?xml version="1.0"?>
 <robot xmlns:xacro="http://www.ros.org/wiki/xacro" name="prbt">
-  <xacro:arg name="robot_prefix" default="prbt_"/>
-  <xacro:arg name="bus_config" default="$(find prbt_robot_support)/config/prbt/bus.yml"/>
-  <xacro:arg name="master_config" default="$(find prbt_robot_support)/config/prbt/master.dcf"/>
-  <xacro:arg name="can_interface" default="vcan0"/>
-  <xacro:arg name="master_bin" default=""/>
-  <xacro:include filename="$(find prbt_robot_support)/urdf/prbt.ros2_control.xacro" />
-  <xacro:include filename="$(find prbt_robot_support)/urdf/prbt_macro.xacro" />
-  <xacro:prbt_ros2_control name="prbt" prefix="$(arg robot_prefix)" bus_config="$(arg bus_config)" master_config="$(arg master_config)" can_interface="$(arg can_interface)" master_bin="$(arg master_bin)" />
-  <!-- TCP Offset -->
-  <xacro:arg name="tcp_offset_xyz" default="0 0 0"/>
-  <xacro:arg name="tcp_offset_rpy" default="0 0 0"/>
-  <!-- instantiate the robot -->
-  <xacro:prbt prefix="$(arg robot_prefix)" />
-  <!-- TCP -->
-  <joint name="$(arg robot_prefix)fixed_joint_tcp" type="fixed">
-    <origin xyz="$(arg tcp_offset_xyz)" rpy="$(arg tcp_offset_rpy)" />
-    <!-- tcp offset from last link -->
-    <parent link="$(arg robot_prefix)flange"/>
-    <child link="$(arg robot_prefix)tcp"/>
-  </joint>
-  <link name="$(arg robot_prefix)tcp" />
+    <xacro:arg name="robot_prefix" default="prbt_"/>
+    <xacro:arg name="bus_config" default="$(find prbt_robot_support)/config/prbt/bus.yml"/>
+    <xacro:arg name="master_config" default="$(find prbt_robot_support)/config/prbt/master.dcf"/>
+    <xacro:arg name="can_interface" default="vcan0"/>
+    <xacro:arg name="master_bin" default=""/>
+    <!-- Import prbt urdf file -->
+    <xacro:include filename="$(find prbt_robot_support)/urdf/prbt_macro.xacro" />
+    <!--xacro:include filename="$(find prbt_robot_support)/urdf/prbt.ros2_control.xacro" /-->
+    <!-- instantiate the robot -->
+    <xacro:prbt prefix="$(arg robot_prefix)" />
+    <link name="world"/>
+    <joint name="world-base_link-fixed" type="fixed">
+        <parent link="world"/>
+        <child link="$(arg robot_prefix)base_link"/>
+    </joint>
 </robot>
