Commit message: separated out description package

File: prbt_description/urdf/prbt_macro.xacro (robot description, xacro)
@@ -19,5 +19,5 @@
         <origin xyz="0 0 0" rpy="0 0 0" />
         <geometry>
-          <mesh filename="package://prbt_robot_support/meshes/foot.dae" />
+          <mesh filename="package://prbt_description/meshes/foot.dae" />
         </geometry>
       </visual>
@@ -48,5 +48,5 @@
         <origin xyz="0 0 0" rpy="0 0 0" />
         <geometry>
-          <mesh filename="package://prbt_robot_support/meshes/link_1.dae" />
+          <mesh filename="package://prbt_description/meshes/link_1.dae" />
         </geometry>
       </visual>
@@ -88,5 +88,5 @@
         <origin xyz="0 0 0" rpy="0 0 0" />
         <geometry>
-          <mesh filename="package://prbt_robot_support/meshes/link_2.dae" />
+          <mesh filename="package://prbt_description/meshes/link_2.dae" />
         </geometry>
       </visual>
@@ -122,5 +122,5 @@
         <origin xyz="0 0 0" rpy="0 0 0" />
         <geometry>
-          <mesh filename="package://prbt_robot_support/meshes/link_3.dae" />
+          <mesh filename="package://prbt_description/meshes/link_3.dae" />
         </geometry>
       </visual>
@@ -162,5 +162,5 @@
         <origin xyz="0 0 0" rpy="0 0 0" />
         <geometry>
-          <mesh filename="package://prbt_robot_support/meshes/link_4.dae" />
+          <mesh filename="package://prbt_description/meshes/link_4.dae" />
         </geometry>
       </visual>
@@ -196,5 +196,5 @@
         <origin xyz="0 0 0" rpy="0 0 0" />
         <geometry>
-          <mesh filename="package://prbt_robot_support/meshes/link_5.dae"/>
+          <mesh filename="package://prbt_description/meshes/link_5.dae"/>
         </geometry>
       </visual>
@@ -249,5 +249,5 @@
         <origin xyz="0 0 0" rpy="0 0 0" />
         <geometry>
-          <mesh filename="package://prbt_robot_support/meshes/flange.dae"/>
+          <mesh filename="package://prbt_description/meshes/flange.dae"/>
         </geometry>
       </visual>
