Commit message: main launch file

File: prbt_description/urdf/prbt.ros2_control.xacro (robot description, xacro)
@@ -18,5 +18,5 @@
         <param name="master_bin">"${master_bin}"</param>
       </hardware>
-      <joint name="prbt_joint_1">
+      <joint name="{prefix}joint_1">
         <param name="node_id">3</param>
         <command_interface name="position"/>

Commit message: update controller spawners

File: prbt_description/urdf/prbt.ros2_control.xacro (robot description, xacro)
@@ -18,5 +18,5 @@
         <param name="master_bin">"${master_bin}"</param>
       </hardware>
-      <joint name="{prefix}joint_1">
+      <joint name="${prefix}joint_1">
         <param name="node_id">3</param>
         <command_interface name="position"/>

File: prbt_robot_moveit_config/config/prbt.urdf.xacro (robot description, xacro)
@@ -8,5 +8,5 @@
     <xacro:arg name="master_bin" default=""/>
     <!-- Import prbt urdf file -->
-    <xacro:include filename="$(find prbt_robot_support)/urdf/prbt_macro.xacro" />
+    <xacro:include filename="$(find prbt_description)/urdf/prbt_macro.xacro" />
     <!-- TCP Offset -->
     <xacro:arg name="tcp_offset_xyz" default="0 0 0"/>

Commit message: update launch config files (#4)

File: prbt_description/urdf/prbt.ros2_control.xacro (robot description, xacro)
@@ -1,70 +1,38 @@
 <?xml version="1.0"?>
 <robot xmlns:xacro="http://www.ros.org/wiki/xacro">
-  <xacro:macro name="prbt_ros2_control" params="
+    <xacro:macro name="prbt_ros2_control" params="
       name
       prefix
       bus_config
       master_config
-      can_interface
-      master_bin
-      initial_positions_file">
-    <xacro:property name="initial_positions" value="${xacro.load_yaml(initial_positions_file)['initial_positions']}"/>
-    <ros2_control name="${name}" type="system">
-      <hardware>
-        <plugin>canopen_ros2_control/Cia402RobotSystem</plugin>
-        <param name="bus_config">${bus_config}</param>
-        <param name="master_config">${master_config}</param>
-        <param name="can_interface_name">${can_interface}</param>
-        <param name="master_bin">"${master_bin}"</param>
-      </hardware>
-      <joint name="${prefix}joint_1">
-        <param name="node_id">3</param>
-        <command_interface name="position"/>
-        <state_interface name="position">
-          <param name="initial_value">${initial_positions['prbt_joint_1']}</param>
-        </state_interface>
-        <state_interface name="velocity"/>
-      </joint>
-      <joint name="${prefix}joint_2">
-        <param name="node_id">4</param>
-        <command_interface name="position"/>
-        <state_interface name="position">
-          <param name="initial_value">${initial_positions['prbt_joint_2']}</param>
-        </state_interface>
-        <state_interface name="velocity"/>
-      </joint>
-      <joint name="${prefix}joint_3">
-        <param name="node_id">5</param>
-        <command_interface name="position"/>
-        <state_interface name="position">
-          <param name="initial_value">${initial_positions['prbt_joint_3']}</param>
-        </state_interface>
-        <state_interface name="velocity"/>
-      </joint>
-      <joint name="${prefix}joint_4">
-        <param name="node_id">6</param>
-        <command_interface name="position"/>
-        <state_interface name="position">
-          <param name="initial_value">${initial_positions['prbt_joint_4']}</param>
-        </state_interface>
-        <state_interface name="velocity"/>
-      </joint>
-      <joint name="${prefix}joint_5">
-        <param name="node_id">7</param>
-        <command_interface name="position"/>
-        <state_interface name="position">
-          <param name="initial_value">${initial_positions['prbt_joint_5']}</param>
-        </state_interface>
-        <state_interface name="velocity"/>
-      </joint>
-      <joint name="${prefix}joint_6">
-        <param name="node_id">8</param>
-        <command_interface name="position"/>
-        <state_interface name="position">
-          <param name="initial_value">${initial_positions['prbt_joint_6']}</param>
-        </state_interface>
-        <state_interface name="velocity"/>
-      </joint>
-    </ros2_control>
-  </xacro:macro>
+      can_interface_name
+      master_bin">
+        <ros2_control name="${name}" type="system">
+            <hardware>
+                <plugin>canopen_ros2_control/RobotSystem</plugin>
+                <param name="bus_config">${bus_config}</param>
+                <param name="master_config">${master_config}</param>
+                <param name="can_interface_name">${can_interface_name}</param>
+                <param name="master_bin">"${master_bin}"</param>
+            </hardware>
+            <joint name="${prefix}joint_1">
+                <param name="device_name">prbt_joint_1</param>
+            </joint>
+            <joint name="${prefix}joint_2">
+                <param name="device_name">prbt_joint_2</param>
+            </joint>
+            <joint name="${prefix}joint_3">
+                <param name="device_name">prbt_joint_3</param>
+            </joint>
+            <joint name="${prefix}joint_4">
+                <param name="device_name">prbt_joint_4</param>
+            </joint>
+            <joint name="${prefix}joint_5">
+                <param name="device_name">prbt_joint_5</param>
+            </joint>
+            <joint name="${prefix}joint_6">
+                <param name="device_name">prbt_joint_6</param>
+            </joint>
+        </ros2_control>
+    </xacro:macro>
 </robot>

File: prbt_description/urdf/prbt.xacro (robot description, xacro)
@@ -1,17 +1,12 @@
 <?xml version="1.0"?>
 <robot xmlns:xacro="http://www.ros.org/wiki/xacro" name="prbt">
-    <xacro:arg name="initial_positions_file" default="$(find prbt_description)/config/initial_positions.yaml" />
     <xacro:arg name="robot_prefix" default="prbt_"/>
     <xacro:arg name="bus_config" default="$(find prbt_robot_support)/config/prbt/bus.yml"/>
     <xacro:arg name="master_config" default="$(find prbt_robot_support)/config/prbt/master.dcf"/>
-    <xacro:arg name="can_interface" default="vcan0"/>
+    <xacro:arg name="can_interface_name" default="vcan0"/>
     <xacro:arg name="master_bin" default=""/>
-    <xacro:arg name="use_ros2_control" default="false"/>
     <!-- Import prbt urdf file -->
     <xacro:include filename="$(find prbt_description)/urdf/prbt_macro.xacro" />
     <xacro:include filename="$(find prbt_description)/urdf/prbt.ros2_control.xacro" />
-    <!-- TCP Offset -->
-    <xacro:arg name="tcp_offset_xyz" default="0 0 0"/>
-    <xacro:arg name="tcp_offset_rpy" default="0 0 0"/>
     <!-- instantiate the robot -->
     <xacro:prbt prefix="$(arg robot_prefix)" />
@@ -21,15 +16,10 @@
         <child link="$(arg robot_prefix)base_link"/>
     </joint>
-    <!-- TCP -->
-    <joint name="$(arg robot_prefix)fixed_joint_tcp" type="fixed">
-        <origin xyz="$(arg tcp_offset_xyz)" rpy="$(arg tcp_offset_rpy)" />
-        <!-- tcp offset from last link -->
-        <parent link="$(arg robot_prefix)flange"/>
-        <child link="$(arg robot_prefix)tcp"/>
-    </joint>
-    <link name="$(arg robot_prefix)tcp" />
-    <!-- ROS2 Control -->
-    <xacro:if value="$(arg use_ros2_control)">
-        <xacro:prbt_ros2_control name="prbt" initial_positions_file="$(arg initial_positions_file)" prefix="$(arg robot_prefix)" bus_config="$(arg bus_config)" master_config="$(arg master_config)" can_interface="$(arg can_interface)" master_bin="$(arg master_bin)"/>
-    </xacro:if>
+    <xacro:prbt_ros2_control
+        name="$(arg robot_prefix)"
+        prefix="$(arg robot_prefix)"
+        bus_config="$(arg bus_config)"
+        master_config="$(arg master_config)"
+        can_interface_name="$(arg can_interface)"
+        master_bin="$(arg master_bin)" />
 </robot>
